File: src/OTHER/MeterMaid Eagle/MeterMaidV2.brd (EAGLE design)
At the start: 74 x 34 mm, 9 parts

Commit message: OTHER additions
Parts:
- removed AP_SW: 5501, switch:5501
- removed C1: 33uf, 50V, rcl:C050-030X075
- removed C2: .01 uf, capacitor-wima:C2.5-3
- removed D1, D2: 1N4004, diode:DO41-10
- removed J1, J2: (no value), con-amp:1X2MTA
- removed SV1: D24V5F5, con-lstb:MA04-1
- added C4: 47uf, rcl:C025-050X050
- added C5, C6: 100nf, rcl:C025-050X050
- added D3, D4: 1N4004, Sam:DO41-10
- added GND, RUN, VIN: (no value), Sam:1X01LP
- added JP3: (no value), Sam:1X04
- U$1: value ESP32DEVKITV1 -> (none); device ESP32-DEVKITV1:ESP32-DEVKITV1 -> ESP32-DEVKITV1MOD:ESP32-DEVKITV2
- moved U$1 3.49 mm to (35.6, 18.7)
Connections:
- removed net 5V_IN: C2.2, SV1.4, U$1.30
- removed net PIN13: D1.A, U$1.28
- removed net PIN25: AP_SW.1A, U$1.23
- removed net RAW_VIN: J2.1
- removed net RUN_GND: J1.1
- removed net VIN: C1.1, D2.C, SV1.2
- new net N$2: C4.2, D3.C, JP3.3
- new net N$4: C5.1, D4.C, RUN.P$1
- new net N$5: C6.2, U$1.16
- new net N$6: D3.A, VIN.P$1
- net GND: now also C4.1, C5.2, C6.1, GND.P$1, JP3.2, U$1.29; no longer AP_SW.NO, C1.2, C2.1, SV1.3, U$1.28
- net N$1: now also JP3.1, U$1.1; no longer D1.C, J1.2
- net N$3: now also D4.A, U$1.28; no longer D2.A, J2.2
Routing:
- net GND: track 0.00 -> 143.5 mm
- net N$1: track 0.00 -> 55.5 mm
- net N$3: track 0.00 -> 46.6 mm
- net N$2: track 0.00 -> 18.5 mm
- net N$5: track 0.00 -> 11.8 mm
- net N$4: track 0.00 -> 11.1 mm
- net N$6: track 0.00 -> 4.07 mm
- added copper zone on layer 16, net GND
