File: OTHER/MeterMaid Eagle/MeterMaid.brd (EAGLE design)
At the start: 74 x 34 mm, 9 parts

Commit message: Updates
Parts:
- added C2: (no value), rcl:C025-050X050
- JP3: value (none) -> D24V5F3
Connections:
- net GND: now also C2.2
- net N$4: now also C2.1
Routing:
- net N$4: track 7.73 -> 10.3 mm
- net GND: track 142.1 -> 142.6 mm
- added copper zone on layer 16, net GND
Changed lines of the file:
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@@
 <grid distance="1" unitdist="mil" unit="mil" style="lines" multiple="10" display="no" altdistance="1" altunitdist="mil" altunit="mil"/>
 <layers>
-<layer number="1" name="Top" color="4" fill="1" visible="no" active="yes"/>
-<layer number="16" name="Bottom" color="1" fill="1" visible="yes" active="yes"/>
-<layer number="17" name="Pads" color="2" fill="1" visible="yes" active="yes"/>
-<layer number="18" name="Vias" color="2" fill="1" visible="no" active="yes"/>
-<layer number="19" name="Unrouted" color="6" fill="1" visible="yes" active="yes"/>
-<layer number="20" name="Dimension" color="24" fill="1" visible="no" active="yes"/>
-<layer number="21" name="tPlace" color="7" fill="1" visible="yes" active="yes"/>
+<layer number="1" name="Top" color="4" fill="1" visible="yes" active="yes"/>
+<layer number="16" name="Bottom" color="21" fill="1" visible="yes" active="yes"/>
+<layer number="17" name="Pads" color="21" fill="1" visible="yes" active="yes"/>
+<layer number="18" name="Vias" color="21" fill="1" visible="yes" active="yes"/>
+<layer number="19" name="Unrouted" color="6" fill="1" visible="no" active="yes"/>
+<layer number="20" name="Dimension" color="24" fill="1" visible="yes" active="yes"/>
+<layer number="21" name="tPlace" color="7" fill="1" visible="no" active="yes"/>
 <layer number="22" name="bPlace" color="7" fill="1" visible="no" active="yes"/>
 <layer number="23" name="tOrigins" color="15" fill="1" visible="no" active="yes"/>
 <layer number="24" name="bOrigins" color="15" fill="1" visible="no" active="yes"/>
-<layer number="25" name="tNames" color="7" fill="1" visible="yes" active="yes"/>
+<layer number="25" name="tNames" color="7" fill="1" visible="no" active="yes"/>
 <layer number="26" name="bNames" color="7" fill="1" visible="no" active="yes"/>
 <layer number="27" name="tValues" color="7" fill="1" visible="no" active="yes"/>
@@
 <layer number="42" name="bRestrict" color="1" fill="10" visible="no" active="yes"/>
 <layer number="43" name="vRestrict" color="2" fill="10" visible="no" active="yes"/>
-<layer number="44" name="Drills" color="7" fill="1" visible="no" active="yes"/>
+<layer number="44" name="Drills" color="49" fill="1" visible="no" active="yes"/>
 <layer number="45" name="Holes" color="7" fill="1" visible="no" active="yes"/>
 <layer number="46" name="Milling" color="3" fill="1" visible="no" active="yes"/>
@@
 <board>
 <plain>
-<wire x1="0" y1="0" x2="74" y2="0" width="0" layer="20"/>
-<wire x1="74" y1="0" x2="74" y2="34" width="0" layer="20"/>
-<wire x1="74" y1="34" x2="0" y2="34" width="0" layer="20"/>
-<wire x1="0" y1="34" x2="0" y2="0" width="0" layer="20"/>
+<wire x1="0" y1="0" x2="74" y2="0" width="0.254" layer="20"/>
+<wire x1="74" y1="0" x2="74" y2="34" width="0.254" layer="20"/>
+<wire x1="74" y1="34" x2="0" y2="34" width="0.254" layer="20"/>
+<wire x1="0" y1="34" x2="0" y2="0" width="0.254" layer="20"/>
 <rectangle x1="56.7354" y1="9.5822" x2="66.9354" y2="22.2822" layer="49"/>
 <circle x="71.992" y="1.952" locked="yes" radius="1.4142125" width="2.25" layer="47"/>
@@
 <elements>
 <element name="U$1" library="ESP32-DEVKITV1MOD" package="ESP32-DEVKITV1" value="ESP32DEVKITV1" x="35.598" y="18.718" locked="yes" smashed="yes"/>
-<element name="JP3" library="pinhead" library_urn="urn:adsk.eagle:library:325" package="1X04" package3d_urn="urn:adsk.eagle:package:22407/2" value="" x="61.9058" y="11.1238" smashed="yes">
+<element name="JP3" library="pinhead" library_urn="urn:adsk.eagle:library:325" package="1X04" package3d_urn="urn:adsk.eagle:package:22407/2" value="D24V5F3" x="61.9058" y="11.1238" smashed="yes">
 <attribute name="NAME" x="56.8766" y="7.9488" size="0.8128" layer="25" ratio="10"/>
 <attribute name="POPULARITY" value="91" x="61.9058" y="11.1238" size="1.778" layer="27" display="off"/>
@@
 <attribute name="POPULARITY" value="64" x="71.628" y="28.194" size="1.778" layer="27" display="off"/>
 <attribute name="VALUE" x="70.358" y="25.019" size="1.27" layer="27"/>
+</element>
+<element name="C2" library="rcl" library_urn="urn:adsk.eagle:library:334" package="C025-050X050" package3d_urn="urn:adsk.eagle:package:23633/1" value="" x="67.1576" y="29.9466" smashed="yes">
+<attribute name="NAME" x="67.5894" y="27.9654" size="1.27" layer="25" ratio="10"/>
+<attribute name="POPULARITY" value="16" x="67.1576" y="29.9466" size="1.778" layer="27" display="off"/>
+<attribute name="SPICEPREFIX" value="C" x="67.1576" y="29.9466" size="1.778" layer="27" display="off"/>
+<attribute name="VALUE" x="64.8716" y="26.1366" size="1.27" layer="27" ratio="10"/>
 </element>
 </elements>
@@
 <wire x1="60.6358" y1="7.874" x2="60.6358" y2="4.8978" width="0.8128" layer="16"/>
 <wire x1="60.6358" y1="4.8978" x2="60.5898" y2="4.8518" width="0.8128" layer="16"/>
-<wire x1="71.628" y1="30.734" x2="70.612" y2="31.75" width="0.8128" layer="16"/>
-<wire x1="71.628" y1="30.734" x2="71.628" y2="28.194" width="0.8128" layer="16"/>
 <wire x1="15.268" y1="5.178" x2="15.268" y2="6.632" width="0.8128" layer="16"/>
 <wire x1="15.268" y1="6.632" x2="16.51" y2="7.874" width="0.8128" layer="16"/>
@@
 <wire x1="15.268" y1="23.7972" x2="17.4752" y2="21.59" width="0.8128" layer="16"/>
 <wire x1="17.4752" y1="21.59" x2="60.6358" y2="21.59" width="0.8128" layer="16"/>
-<wire x1="60.6358" y1="21.59" x2="60.6358" y2="29.8696" width="0.8128" layer="16"/>
-<wire x1="60.5536" y1="29.9518" x2="60.549" y2="29.9564" width="0.8128" layer="16"/>
-<wire x1="70.612" y1="31.75" x2="64.516" y2="31.75" width="0.8128" layer="16"/>
-<wire x1="64.516" y1="31.75" x2="61.1632" y2="31.75" width="0.8128" layer="16"/>
-<wire x1="61.1632" y1="31.75" x2="60.5536" y2="31.1404" width="0.8128" layer="16"/>
-<wire x1="60.5536" y1="31.1404" x2="60.5536" y2="29.9518" width="0.8128" layer="16"/>
-<wire x1="60.5536" y1="29.9518" x2="60.6358" y2="29.8696" width="0.8128" layer="16"/>
+<wire x1="60.6358" y1="29.8696" x2="60.6358" y2="21.59" width="0.8128" layer="16"/>
 <wire x1="60.6358" y1="7.874" x2="60.6358" y2="11.1238" width="0.8128" layer="16"/>
 <wire x1="60.6358" y1="21.59" x2="60.6358" y2="11.1238" width="0.8128" layer="16"/>
-<wire x1="64.516" y1="30.035" x2="64.516" y2="31.75" width="0.8128" layer="16"/>
+<contactref element="C2" pad="2"/>
+<polygon width="0.0762" layer="16" isolate="0.6096">
+<vertex x="0.0254" y="33.9852"/>
+<vertex x="73.9902" y="33.9852"/>
+<vertex x="73.9902" y="0.0254"/>
+<vertex x="0.0254" y="0.0254"/>
+</polygon>
+<wire x1="60.549" y1="29.9564" x2="60.6358" y2="29.8696" width="0.1524" layer="16"/>
+<wire x1="60.549" y1="29.9564" x2="62.876" y2="32.2834" width="0.8128" layer="16"/>
+<wire x1="70.3072" y1="32.2834" x2="68.4276" y2="32.2834" width="0.8128" layer="16"/>
+<wire x1="68.4276" y1="32.2834" x2="62.876" y2="32.2834" width="0.8128" layer="16"/>
+<wire x1="71.628" y1="28.194" x2="71.628" y2="30.9626" width="0.8128" layer="16"/>
+<wire x1="71.628" y1="30.9626" x2="70.3072" y2="32.2834" width="0.8128" layer="16"/>
+<wire x1="68.4276" y1="29.9466" x2="68.4276" y2="32.2834" width="0.8128" layer="16"/>
 </signal>
 <signal name="N$2">
@@
 <contactref element="D2" pad="C"/>
 <contactref element="RUN" pad="1"/>
-<wire x1="67.332" y1="24.586" x2="69.088" y2="24.586" width="0.8128" layer="16"/>
-<wire x1="69.088" y1="24.586" x2="71.576" y2="24.586" width="0.8128" layer="16"/>
+<wire x1="67.332" y1="24.586" x2="71.576" y2="24.586" width="0.8128" layer="16"/>
 <wire x1="71.576" y1="24.586" x2="71.628" y2="24.638" width="0.8128" layer="16"/>
-<wire x1="69.088" y1="28.003" x2="69.088" y2="24.586" width="0.8128" layer="16"/>
+<contactref element="C2" pad="1"/>
+<wire x1="65.8876" y1="29.9466" x2="65.8876" y2="27.8384" width="0.8128" layer="16"/>
+<wire x1="67.3354" y1="26.3906" x2="65.8876" y2="27.8384" width="0.8128" layer="16"/>
+<wire x1="67.332" y1="24.586" x2="67.332" y2="26.3872" width="0.8128" layer="16"/>
+<wire x1="67.332" y1="26.3872" x2="67.3354" y2="26.3906" width="0.8128" layer="16"/>
 </signal>
 <signal name="N$5">
@@
 <signal name="N$8">
 <via x="60.5536" y="29.9466" extent="1-16" drill="0.35" diameter="1.3"/>
-</signal>
-<signal name="N$9">
-<via x="67.1068" y="29.9974" extent="1-16" drill="0.35" diameter="1.3"/>
-<via x="64.5414" y="29.972" extent="1-16" drill="0.35" diameter="1.3"/>
-<wire x1="64.5414" y1="29.972" x2="67.1068" y2="29.9974" width="0" layer="19" extent="1-1"/>
 </signal>
 <signal name="N$10">
@@
 <mfgpreviewcolor name="substratecolor" color="0xFF786E46"/>
 </mfgpreviewcolors>
+<errors>
+</errors>
 </board>
 </drawing>
